File: Hardware/Production/Qwiic_High_Performance_Magnetometer_X01-Panel.brd (EAGLE design)
At the start: 123.2 x 117.3 mm, 1078 parts, among them J1 Qwiic, J10 Qwiic, J13 Qwiic, J14 Qwiic, J17 Qwiic, J18 Qwiic, J2 Qwiic, J21 Qwiic, J22 Qwiic, J25 Qwiic, J26 Qwiic, J29 Qwiic, J30 Qwiic, J33 Qwiic, J34 Qwiic, J37 Qwiic, J38 Qwiic, J41 Qwiic, J42 Qwiic, J45 Qwiic, J46 Qwiic, J49 Qwiic, J5 Qwiic, J50 Qwiic, J53 Qwiic, J54 Qwiic, J57 Qwiic, J58 Qwiic, J6 Qwiic, J61 Qwiic, J62 Qwiic, J9 Qwiic, U1 MMC5893MA_QFN16, U10 MMC5893MA_QFN16, U11 MMC5893MA_QFN16, U12 MMC5893MA_QFN16, U13 MMC5893MA_QFN16, U14 MMC5893MA_QFN16, U15 MMC5893MA_QFN16, U16 MMC5893MA_QFN16, U2 MMC5893MA_QFN16, U3 MMC5893MA_QFN16, U4 MMC5893MA_QFN16, U5 MMC5893MA_QFN16, U6 MMC5893MA_QFN16, U7 MMC5893MA_QFN16, U8 MMC5893MA_QFN16, U9 MMC5893MA_QFN16

Commit message: Added production files; updated BOM.
Parts:
- added U$641: (no value), output:HIGH_PERFORMANCE11
- added U$642: (no value), output:MAGNETOMETER12
- added U$643: (no value), output:#GND#4
- added U$644: (no value), output:#3#3V#0
- added U$645: (no value), output:#COPI#12
- added U$646: (no value), output:#CIPO#11
- added U$647: (no value), output:#SCK#13
- added U$648: (no value), output:##CS##10
- added U$649: SPARKX-LOGO2, SparkX:SPARKX-TINY
- added U$650: SPARKX-LOGO3, SparkX:SPARKX-SMALL
- added U$651: (no value), output:MADE_IN_THE_USA20
- added U$652: (no value), output:#SCL#6
- added U$653: (no value), output:#SDA#5
- added U$654: (no value), output:Z17
- added U$655, U$656: (no value), SER:MMC5983MA0
- U$100, U$223: device output:Y16 -> output:##CS##10
- U$101, U$142, U$581, U$622: device output:X15 -> output:#3#3V#0
- U$102, U$61: device output:X15 -> output:Y16
- U$103, U$63: device output:Y16 -> output:X15
- U$104, U$144: device output:Z17 -> output:X15
- U$105, U$225, U$228, U$348: device output:#GND#4 -> output:Y16
- U$106, U$285: device output:HIGH_PERFORMANCE11 -> output:Z17
- U$107, U$166: device output:MAGNETOMETER12 -> output:#GND#4
- U$108, U$128: device output:#GND#4 -> output:HIGH_PERFORMANCE11
- U$109, U$47, U$539, U$601: device output:#3#3V#0 -> output:MAGNETOMETER12
- U$110, U$230, U$336, U$576: device output:#COPI#12 -> output:#GND#4
- U$111, U$335, U$511, U$575: device output:#CIPO#11 -> output:#3#3V#0
- U$112, U$57: device output:#SCK#13 -> output:#COPI#12
- U$113, U$138: device output:##CS##10 -> output:#CIPO#11
- U$114: value SPARKX-LOGO2 -> (none); device SparkX:SPARKX-TINY -> output:#SCK#13
- U$115: value SPARKX-LOGO3 -> (none); device SparkX:SPARKX-SMALL -> output:##CS##10
- U$116: value (none) -> SPARKX-LOGO2; device output:MADE_IN_THE_USA20 -> SparkX:SPARKX-TINY
- U$117: value (none) -> SPARKX-LOGO3; device output:#SCL#6 -> SparkX:SPARKX-SMALL
- U$118: device output:#SDA#5 -> output:MADE_IN_THE_USA20
- U$119, U$464: device output:Z17 -> output:#SCL#6
- U$120: device numbers:PCB#163280 -> output:#SDA#5
- U$121, U$229, U$367: device output:#3#3V#0 -> output:Z17
- U$122, U$328, U$368, U$42, U$82: device output:#GND#4 -> SER:MMC5983MA0
- U$123, U$163, U$369, U$409: device output:#INT#7 -> SER:MMC5983MA0
- U$124: device output:PWR9 -> output:#3#3V#0
- U$125, U$66: device output:HIGH_PERFORMANCE11 -> output:#GND#4
- U$126: device output:MAGNETOMETER12 -> output:#INT#7
- U$127, U$619: device output:#3#3V#0 -> output:PWR9
- U$129: device output:#INT#7 -> output:MAGNETOMETER12
- U$130, U$370: device output:#LED#8 -> output:#3#3V#0
- U$131, U$371: device output:#I2C#9 -> output:#GND#4
- U$132, U$372: device output:#SPI#9 -> output:#INT#7
- U$133: device output:#SCL#6 -> output:#LED#8
- U$134: device output:#SDA#5 -> output:#I2C#9
- U$135: device output:#CIPO#11 -> output:#SPI#9
- U$136: device output:#COPI#12 -> output:#SCL#6
- U$137: device output:#SCK#13 -> output:#SDA#5
- U$139, U$481, U$549: device output:#3#3V#0 -> output:#COPI#12
- U$140, U$263: device output:Y16 -> output:#SCK#13
- U$141, U$182: device output:X15 -> output:##CS##10
- U$145, U$185, U$268, U$308: device output:#GND#4 -> output:X15
- U$146, U$266: device output:HIGH_PERFORMANCE11 -> output:Y16
- U$147, U$326: device output:MAGNETOMETER12 -> output:Z17
- U$149, U$579, U$87: device output:#3#3V#0 -> output:HIGH_PERFORMANCE11
- U$150, U$416: device output:#COPI#12 -> output:MAGNETOMETER12
- U$151, U$271, U$295, U$535: device output:#CIPO#11 -> output:#GND#4
- U$152, U$417, U$552: device output:#SCK#13 -> output:#3#3V#0
- U$153, U$98: device output:##CS##10 -> output:#COPI#12
- U$154: value SPARKX-LOGO2 -> (none); device SparkX:SPARKX-TINY -> output:#CIPO#11
- U$155: value SPARKX-LOGO3 -> (none); device SparkX:SPARKX-SMALL -> output:#SCK#13
- U$156: device output:MADE_IN_THE_USA20 -> output:##CS##10
- U$157: value (none) -> SPARKX-LOGO2; device output:#SCL#6 -> SparkX:SPARKX-TINY
- U$158: value (none) -> SPARKX-LOGO3; device output:#SDA#5 -> SparkX:SPARKX-SMALL
- U$159: device output:Z17 -> output:MADE_IN_THE_USA20
- U$160: device numbers:PCB#163280 -> output:#SCL#6
- U$161, U$219, U$407, U$629: device output:#3#3V#0 -> output:#SDA#5
- U$162, U$188, U$408, U$65: device output:#GND#4 -> output:Z17
- U$164, U$204: device output:PWR9 -> SER:MMC5983MA0
- U$165, U$306: device output:HIGH_PERFORMANCE11 -> output:#3#3V#0
- U$167, U$419: device output:#3#3V#0 -> output:#INT#7
- U$168: device output:#GND#4 -> output:PWR9
- U$169: device output:#INT#7 -> output:HIGH_PERFORMANCE11
- U$170: device output:#LED#8 -> output:MAGNETOMETER12
- U$171, U$411: device output:#I2C#9 -> output:#3#3V#0
- U$172, U$412: device output:#SPI#9 -> output:#GND#4
- U$173, U$413: device output:#SCL#6 -> output:#INT#7
- U$174: device output:#SDA#5 -> output:#LED#8
- U$175: device output:#CIPO#11 -> output:#I2C#9
- U$176: device output:#COPI#12 -> output:#SPI#9
- U$177: device output:#SCK#13 -> output:#SCL#6
- U$178: device output:##CS##10 -> output:#SDA#5
- U$179, U$441, U$589: device output:#3#3V#0 -> output:#CIPO#11
- U$180, U$303: device output:Y16 -> output:#COPI#12
- U$181, U$222: device output:X15 -> output:#SCK#13
- U$183, U$540, U$60: device output:Y16 -> output:#3#3V#0
- U$184, U$64: device output:Z17 -> output:Y16
- U$186, U$226: device output:HIGH_PERFORMANCE11 -> output:X15
- U$187, U$307: device output:MAGNETOMETER12 -> output:Y16
- U$189, U$207, U$459, U$561, U$69: device output:#3#3V#0 -> output:#GND#4
- U$190, U$456: device output:#COPI#12 -> output:HIGH_PERFORMANCE11
- U$191, U$375: device output:#CIPO#11 -> output:MAGNETOMETER12
- U$192, U$312, U$377, U$617: device output:#SCK#13 -> output:#GND#4
- U$193, U$458, U$593: device output:##CS##10 -> output:#3#3V#0
- U$194: value SPARKX-LOGO2 -> (none); device SparkX:SPARKX-TINY -> output:#COPI#12
- U$195: value SPARKX-LOGO3 -> (none); device SparkX:SPARKX-SMALL -> output:#CIPO#11
- U$196: device output:MADE_IN_THE_USA20 -> output:#SCK#13
- U$197: device output:#SCL#6 -> output:##CS##10
- U$198: value (none) -> SPARKX-LOGO2; device output:#SDA#5 -> SparkX:SPARKX-TINY
- U$199: value (none) -> SPARKX-LOGO3; device output:Z17 -> SparkX:SPARKX-SMALL
- U$200: device numbers:PCB#163280 -> output:MADE_IN_THE_USA20
- U$201, U$259, U$447: device output:#3#3V#0 -> output:#SCL#6
- U$202, U$448, U$465, U$588: device output:#GND#4 -> output:#SDA#5
- U$203, U$449: device output:#INT#7 -> output:Z17
- U$205, U$245: device output:HIGH_PERFORMANCE11 -> SER:MMC5983MA0
- U$206, U$347: device output:MAGNETOMETER12 -> output:#3#3V#0
- U$208: device output:#GND#4 -> output:#INT#7
- U$209: device output:#INT#7 -> output:PWR9
- U$210: device output:#LED#8 -> output:HIGH_PERFORMANCE11
- U$211: device output:#I2C#9 -> output:MAGNETOMETER12
- U$212, U$452: device output:#SPI#9 -> output:#3#3V#0
- U$213, U$397, U$453, U$517: device output:#SCL#6 -> output:#GND#4
- U$214, U$454: device output:#SDA#5 -> output:#INT#7
- U$215: device output:#CIPO#11 -> output:#LED#8
- U$216: device output:#COPI#12 -> output:#I2C#9
- U$217: device output:#SCK#13 -> output:#SPI#9
- U$218: device output:##CS##10 -> output:#SCL#6
- U$220, U$343: device output:Y16 -> output:#CIPO#11
- U$221, U$262: device output:X15 -> output:#COPI#12
- U$224, U$439: device output:Z17 -> output:#3#3V#0
- U$227, U$267: device output:MAGNETOMETER12 -> output:X15
- U$231, U$415: device output:#CIPO#11 -> output:HIGH_PERFORMANCE11
- U$232, U$457: device output:#SCK#13 -> output:MAGNETOMETER12
- U$233, U$353, U$418: device output:##CS##10 -> output:#GND#4
- U$234, U$634: value SPARKX-LOGO2 -> (none); device SparkX:SPARKX-TINY -> output:#3#3V#0
- U$235: value SPARKX-LOGO3 -> (none); device SparkX:SPARKX-SMALL -> output:#COPI#12
- U$236: device output:MADE_IN_THE_USA20 -> output:#CIPO#11
- U$237: device output:#SCL#6 -> output:#SCK#13
- U$238: device output:#SDA#5 -> output:##CS##10
- U$239: value (none) -> SPARKX-LOGO2; device output:Z17 -> SparkX:SPARKX-TINY
- U$240: value (none) -> SPARKX-LOGO3; device numbers:PCB#163280 -> SparkX:SPARKX-SMALL
- U$241, U$487: device output:#3#3V#0 -> output:MADE_IN_THE_USA20
- U$242, U$488, U$505, U$628: device output:#GND#4 -> output:#SCL#6
- U$243, U$489: device output:#INT#7 -> output:#SDA#5
- U$244: device output:PWR9 -> output:Z17
- U$246, U$286: device output:MAGNETOMETER12 -> SER:MMC5983MA0
- U$250: device output:#LED#8 -> output:PWR9
- U$251: device output:#I2C#9 -> output:HIGH_PERFORMANCE11
- U$252: device output:#SPI#9 -> output:MAGNETOMETER12
- U$253, U$357, U$493: device output:#SCL#6 -> output:#3#3V#0
- U$254, U$438, U$494, U$558: device output:#SDA#5 -> output:#GND#4
- U$255, U$495: device output:#CIPO#11 -> output:#INT#7
- U$256: device output:#COPI#12 -> output:#LED#8
- U$257: device output:#SCK#13 -> output:#I2C#9
- U$258: device output:##CS##10 -> output:#SPI#9
- U$260, U$383: device output:Y16 -> output:#SDA#5
- U$261, U$302: device output:X15 -> output:#CIPO#11
- U$264, U$279: device output:Z17 -> output:##CS##10
- U$265, U$288, U$388, U$48, U$562: device output:#GND#4 -> output:#3#3V#0
- U$269, U$389: device output:#3#3V#0 -> output:Y16
- U$270: device output:#COPI#12 -> output:Z17
- U$272, U$497: device output:#SCK#13 -> output:HIGH_PERFORMANCE11
- U$273, U$498: device output:##CS##10 -> output:MAGNETOMETER12
- U$274, U$394: value SPARKX-LOGO2 -> (none); device SparkX:SPARKX-TINY -> output:#GND#4
- U$275: value SPARKX-LOGO3 -> (none); device SparkX:SPARKX-SMALL -> output:#3#3V#0
- U$276: device output:MADE_IN_THE_USA20 -> output:#COPI#12
- U$277: device output:#SCL#6 -> output:#CIPO#11
- U$278: device output:#SDA#5 -> output:#SCK#13
- U$280: value (none) -> SPARKX-LOGO2; device numbers:PCB#163280 -> SparkX:SPARKX-TINY
- U$281, U$527: value (none) -> SPARKX-LOGO3; device output:#3#3V#0 -> SparkX:SPARKX-SMALL
- U$282, U$528: device output:#GND#4 -> output:MADE_IN_THE_USA20
- U$283, U$529: device output:#INT#7 -> output:#SCL#6
- U$284: device output:PWR9 -> output:#SDA#5
- U$287, U$327, U$41, U$81: device output:#3#3V#0 -> SER:MMC5983MA0
- U$289, U$43, U$49: device output:#INT#7 -> output:#GND#4
- U$290, U$50: device output:#LED#8 -> output:#INT#7
- U$291: device output:#I2C#9 -> output:PWR9
- U$292: device output:#SPI#9 -> output:HIGH_PERFORMANCE11
- U$293, U$437: device output:#SCL#6 -> output:MAGNETOMETER12
- U$294, U$398, U$534: device output:#SDA#5 -> output:#3#3V#0
- U$296, U$536: device output:#COPI#12 -> output:#INT#7
- U$297: device output:#SCK#13 -> output:#LED#8
- U$298: device output:##CS##10 -> output:#I2C#9
- U$299: device output:#3#3V#0 -> output:#SPI#9
- U$300, U$423: device output:Y16 -> output:#SCL#6
- U$301, U$342: device output:X15 -> output:#SDA#5
- U$304, U$319: device output:Z17 -> output:#SCK#13
- U$305, U$402, U$428: device output:#GND#4 -> output:##CS##10
- U$309, U$349: device output:#3#3V#0 -> output:X15
- U$310, U$430: device output:#COPI#12 -> output:Y16
- U$311: device output:#CIPO#11 -> output:Z17
- U$313, U$538: device output:##CS##10 -> output:HIGH_PERFORMANCE11
- U$314: value SPARKX-LOGO2 -> (none); device SparkX:SPARKX-TINY -> output:MAGNETOMETER12
- U$315, U$435: value SPARKX-LOGO3 -> (none); device SparkX:SPARKX-SMALL -> output:#GND#4
- U$316: device output:MADE_IN_THE_USA20 -> output:#3#3V#0
- U$317: device output:#SCL#6 -> output:#COPI#12
- U$318: device output:#SDA#5 -> output:#CIPO#11
- U$320: device numbers:PCB#163280 -> output:##CS##10
- U$321, U$567: value (none) -> SPARKX-LOGO2; device output:#3#3V#0 -> SparkX:SPARKX-TINY
- U$322, U$568: value (none) -> SPARKX-LOGO3; device output:#GND#4 -> SparkX:SPARKX-SMALL
- U$323, U$569: device output:#INT#7 -> output:MADE_IN_THE_USA20
- U$324: device output:PWR9 -> output:#SCL#6
- U$325, U$506: device output:HIGH_PERFORMANCE11 -> output:#SDA#5
- U$329, U$603, U$83, U$89: device output:#INT#7 -> output:#3#3V#0
- U$330, U$90: device output:#LED#8 -> output:#GND#4
- U$331, U$91: device output:#I2C#9 -> output:#INT#7
- U$332: device output:#SPI#9 -> output:PWR9
- U$333, U$477: device output:#SCL#6 -> output:HIGH_PERFORMANCE11
- U$334, U$478: device output:#SDA#5 -> output:MAGNETOMETER12
- U$337, U$577: device output:#SCK#13 -> output:#INT#7
- U$338: device output:##CS##10 -> output:#LED#8
- U$339: device output:#3#3V#0 -> output:#I2C#9
- U$340, U$463: device output:Y16 -> output:#SPI#9
- U$341, U$382: device output:X15 -> output:#SCL#6
- U$344, U$399: device output:Z17 -> output:#COPI#12
- U$345, U$442, U$468: device output:#GND#4 -> output:#SCK#13
- U$346, U$525: device output:HIGH_PERFORMANCE11 -> output:##CS##10
- U$350, U$390: device output:#COPI#12 -> output:X15
- U$351, U$471: device output:#CIPO#11 -> output:Y16
- U$352: device output:#SCK#13 -> output:Z17
- U$354: value SPARKX-LOGO2 -> (none); device SparkX:SPARKX-TINY -> output:HIGH_PERFORMANCE11
- U$355: value SPARKX-LOGO3 -> (none); device SparkX:SPARKX-SMALL -> output:MAGNETOMETER12
- U$356, U$476: device output:MADE_IN_THE_USA20 -> output:#GND#4
- U$358: device output:#SDA#5 -> output:#COPI#12
- U$359, U$384: device output:Z17 -> output:#CIPO#11
- U$360: device numbers:PCB#163280 -> output:#SCK#13
- U$361, U$469, U$59, U$607: device output:#3#3V#0 -> output:##CS##10
- U$362, U$608: value (none) -> SPARKX-LOGO2; device output:#GND#4 -> SparkX:SPARKX-TINY
- U$363, U$609: value (none) -> SPARKX-LOGO3; device output:#INT#7 -> SparkX:SPARKX-SMALL
- U$364: device output:PWR9 -> output:MADE_IN_THE_USA20
- U$365, U$546: device output:HIGH_PERFORMANCE11 -> output:#SCL#6
- U$366, U$547: device output:MAGNETOMETER12 -> output:#SDA#5
- U$373: device output:#SCL#6 -> output:PWR9
- U$374, U$518: device output:#SDA#5 -> output:HIGH_PERFORMANCE11
- U$376, U$470, U$616, U$70: device output:#COPI#12 -> output:#3#3V#0
- U$378, U$618: device output:##CS##10 -> output:#INT#7
- U$379: device output:#3#3V#0 -> output:#LED#8
- U$380, U$503: device output:Y16 -> output:#I2C#9
- U$381, U$422: device output:X15 -> output:#SPI#9
- U$385, U$508, U$522: device output:#GND#4 -> output:#COPI#12
- U$386, U$565: device output:HIGH_PERFORMANCE11 -> output:#SCK#13
- U$387, U$566: device output:MAGNETOMETER12 -> output:##CS##10
- U$391, U$431: device output:#CIPO#11 -> output:X15
- U$392, U$512: device output:#SCK#13 -> output:Y16
- U$393: device output:##CS##10 -> output:Z17
- U$395: value SPARKX-LOGO3 -> (none); device SparkX:SPARKX-SMALL -> output:HIGH_PERFORMANCE11
- U$396: device output:MADE_IN_THE_USA20 -> output:MAGNETOMETER12
- U$40, U$480: device numbers:PCB#163280 -> output:#3#3V#0
- U$400: device numbers:PCB#163280 -> output:#CIPO#11
- U$401, U$509, U$99: device output:#3#3V#0 -> output:#SCK#13
- U$403: value (none) -> SPARKX-LOGO2; device output:#INT#7 -> SparkX:SPARKX-TINY
- U$404: value (none) -> SPARKX-LOGO3; device output:PWR9 -> SparkX:SPARKX-SMALL
- U$405: device output:HIGH_PERFORMANCE11 -> output:MADE_IN_THE_USA20
- U$406, U$587: device output:MAGNETOMETER12 -> output:#SCL#6
- U$410, U$450: device output:#LED#8 -> SER:MMC5983MA0
- U$414: device output:#SDA#5 -> output:PWR9
- U$420, U$543: device output:Y16 -> output:#LED#8
- U$421, U$462: device output:X15 -> output:#I2C#9
- U$424, U$79: device output:Z17 -> output:#SDA#5
- U$425, U$482, U$548: device output:#GND#4 -> output:#CIPO#11
- U$426: device output:HIGH_PERFORMANCE11 -> output:#COPI#12
- U$427, U$606: device output:MAGNETOMETER12 -> output:#SCK#13
- U$432, U$472: device output:#SCK#13 -> output:X15
- U$433, U$553: device output:##CS##10 -> output:Y16
- U$434: value SPARKX-LOGO2 -> (none); device SparkX:SPARKX-TINY -> output:Z17
- U$436: device output:MADE_IN_THE_USA20 -> output:HIGH_PERFORMANCE11
- U$44: device output:PWR9 -> output:#INT#7
- U$440: device numbers:PCB#163280 -> output:#COPI#12
- U$443: device output:#INT#7 -> output:##CS##10
- U$444: value (none) -> SPARKX-LOGO2; device output:PWR9 -> SparkX:SPARKX-TINY
- U$445: value (none) -> SPARKX-LOGO3; device output:HIGH_PERFORMANCE11 -> SparkX:SPARKX-SMALL
- U$446: device output:MAGNETOMETER12 -> output:MADE_IN_THE_USA20
- U$45: device output:HIGH_PERFORMANCE11 -> output:PWR9
- U$451, U$491: device output:#I2C#9 -> SER:MMC5983MA0
- U$455: device output:#CIPO#11 -> output:PWR9
- U$46, U$67: device output:MAGNETOMETER12 -> output:HIGH_PERFORMANCE11
- U$460, U$583: device output:Y16 -> output:#INT#7
- U$461, U$502: device output:X15 -> output:#LED#8
- U$466, U$605: device output:HIGH_PERFORMANCE11 -> output:#CIPO#11
- U$467: device output:MAGNETOMETER12 -> output:#COPI#12
- U$473, U$513: device output:##CS##10 -> output:X15
- U$474, U$594: value SPARKX-LOGO2 -> (none); device SparkX:SPARKX-TINY -> output:Y16
- U$475: value SPARKX-LOGO3 -> (none); device SparkX:SPARKX-SMALL -> output:Z17
- U$479, U$599: device output:Z17 -> output:#GND#4
- U$483: device output:#INT#7 -> output:#SCK#13
- U$484: device output:PWR9 -> output:##CS##10
- U$485: value (none) -> SPARKX-LOGO2; device output:HIGH_PERFORMANCE11 -> SparkX:SPARKX-TINY
- U$486: value (none) -> SPARKX-LOGO3; device output:MAGNETOMETER12 -> SparkX:SPARKX-SMALL
- U$490: device output:#LED#8 -> output:Z17
- U$492, U$532: device output:#SPI#9 -> SER:MMC5983MA0
- U$496: device output:#COPI#12 -> output:PWR9
- U$500, U$623: device output:Y16 -> output:#GND#4
- U$501, U$542: device output:X15 -> output:#INT#7
- U$504: device output:Z17 -> output:#SPI#9
- U$507: device output:MAGNETOMETER12 -> output:#CIPO#11
- U$51: device output:#I2C#9 -> output:#LED#8
- U$510: device output:#COPI#12 -> output:##CS##10
- U$514, U$554: value SPARKX-LOGO2 -> (none); device SparkX:SPARKX-TINY -> output:X15
- U$515, U$635: value SPARKX-LOGO3 -> (none); device SparkX:SPARKX-SMALL -> output:Y16
- U$516: device output:MADE_IN_THE_USA20 -> output:Z17
- U$519: device output:Z17 -> output:MAGNETOMETER12
- U$52: device output:#SPI#9 -> output:#I2C#9
- U$520, U$640: device numbers:PCB#163280 -> output:#GND#4
- U$523: device output:#INT#7 -> output:#CIPO#11
- U$524: device output:PWR9 -> output:#SCK#13
- U$526: value (none) -> SPARKX-LOGO2; device output:MAGNETOMETER12 -> SparkX:SPARKX-TINY
- U$53: device output:#SCL#6 -> output:#SPI#9
- U$530: device output:#LED#8 -> output:#SDA#5
- U$531: device output:#I2C#9 -> output:Z17
- U$533, U$573: device output:#SCL#6 -> SER:MMC5983MA0
- U$537: device output:#SCK#13 -> output:PWR9
- U$54, U$78: device output:#SDA#5 -> output:#SCL#6
- U$541, U$582: device output:X15 -> output:#GND#4
- U$544: device output:Z17 -> output:#I2C#9
- U$545: device output:#GND#4 -> output:#SPI#9
- U$55: device output:#CIPO#11 -> output:#SDA#5
- U$550: device output:#COPI#12 -> output:#SCK#13
- U$551: device output:#CIPO#11 -> output:##CS##10
- U$555, U$595: value SPARKX-LOGO3 -> (none); device SparkX:SPARKX-SMALL -> output:X15
- U$556: device output:MADE_IN_THE_USA20 -> output:Y16
- U$557, U$613: device output:#SCL#6 -> output:Z17
- U$559: device output:Z17 -> output:HIGH_PERFORMANCE11
- U$56, U$630: device output:#COPI#12 -> output:#CIPO#11
- U$560: device numbers:PCB#163280 -> output:MAGNETOMETER12
- U$563: device output:#INT#7 -> output:#COPI#12
- U$564: device output:PWR9 -> output:#CIPO#11
- U$570: device output:#LED#8 -> output:#SCL#6
- U$571: device output:#I2C#9 -> output:#SDA#5
- U$572: device output:#SPI#9 -> output:Z17
- U$574, U$614: device output:#SDA#5 -> SER:MMC5983MA0
- U$578: device output:##CS##10 -> output:PWR9
- U$58, U$73: device output:##CS##10 -> output:#SCK#13
- U$580: device output:Y16 -> output:MAGNETOMETER12
- U$584: device output:Z17 -> output:#LED#8
- U$585: device output:#GND#4 -> output:#I2C#9
- U$586: device output:HIGH_PERFORMANCE11 -> output:#SPI#9
- U$591: device output:#CIPO#11 -> output:#SCK#13
- U$592: device output:#SCK#13 -> output:##CS##10
- U$596, U$636: device output:MADE_IN_THE_USA20 -> output:X15
- U$597: device output:#SCL#6 -> output:Y16
- U$598: device output:#SDA#5 -> output:Z17
- U$600: device numbers:PCB#163280 -> output:HIGH_PERFORMANCE11
- U$604: device output:PWR9 -> output:#COPI#12
- U$610: device output:#LED#8 -> output:MADE_IN_THE_USA20
- U$611: device output:#I2C#9 -> output:#SCL#6
- U$612: device output:#SPI#9 -> output:#SDA#5
- U$615: device output:#CIPO#11 -> SER:MMC5983MA0
- U$620: device output:Y16 -> output:HIGH_PERFORMANCE11
- U$621: device output:X15 -> output:MAGNETOMETER12
- U$624: device output:Z17 -> output:#INT#7
- U$625: device output:#GND#4 -> output:#LED#8
- U$626: device output:HIGH_PERFORMANCE11 -> output:#I2C#9
- U$627: device output:MAGNETOMETER12 -> output:#SPI#9
- U$631, U$71: device output:#CIPO#11 -> output:#COPI#12
- U$637: device output:#SCL#6 -> output:X15
- U$638: device output:#SDA#5 -> output:Y16
- U$68, U$88: device output:#GND#4 -> output:MAGNETOMETER12
- U$72, U$97: device output:#SCK#13 -> output:#CIPO#11
- U$74: value SPARKX-LOGO2 -> (none); device SparkX:SPARKX-TINY -> output:##CS##10
- U$75: value SPARKX-LOGO3 -> SPARKX-LOGO2; device SparkX:SPARKX-SMALL -> SparkX:SPARKX-TINY
- U$76: value (none) -> SPARKX-LOGO3; device output:MADE_IN_THE_USA20 -> SparkX:SPARKX-SMALL
- U$77: device output:#SCL#6 -> output:MADE_IN_THE_USA20
- U$80: device numbers:PCB#163280 -> output:Z17
- U$84: device output:PWR9 -> output:#GND#4
- U$85: device output:HIGH_PERFORMANCE11 -> output:#INT#7
- U$86: device output:MAGNETOMETER12 -> output:PWR9
- U$92: device output:#SPI#9 -> output:#LED#8
- U$93: device output:#SCL#6 -> output:#I2C#9
- U$94: device output:#SDA#5 -> output:#SPI#9
- U$95: device output:#CIPO#11 -> output:#SCL#6
- U$96: device output:#COPI#12 -> output:#SDA#5
- moved U$484 103.2 mm to (96.8, 53.5), flipped to the bottom, turned to 270 degrees
- moved U$483 99.0 mm to (94.2, 53.5), flipped to the bottom
- moved U$490 98.1 mm to (98.4, 56.6), flipped to the top
- moved U$164 93.6 mm to (90.3, 11.2), flipped to the bottom
- moved U$162 92.3 mm to (98.4, 4.83), turned to 0 degrees
- moved U$326 90.7 mm to (98.4, 30.7)
- moved U$324 90.1 mm to (90.4, 49.7), flipped to the bottom, turned to 270 degrees
- moved U$163 89.6 mm to (90.4, 15.5), turned to 0 degrees
- moved U$481 88.1 mm to (89.2, 53.5), flipped to the bottom
- moved U$482 88.1 mm to (91.7, 53.5), flipped to the bottom
- moved U$489 84.3 mm to (87.9, 75.6)
- moved U$327 82.6 mm to (90.4, 41.4), flipped to the top, turned to 0 degrees
- moved U$328 82.1 mm to (90.3, 37.1), turned to 0 degrees
- moved U$491 82.1 mm to (90.4, 67.3), flipped to the top
- moved U$322 81.2 mm to (90.7, 39.9), flipped to the bottom, turned to 0 degrees
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Routing:
- net SDA/COPI8: track 42.8 -> 51.8 mm
- net SDA/COPI9: track 42.8 -> 51.8 mm
- net SDA/COPI10: track 42.8 -> 51.8 mm
- net SDA/COPI1: track 42.8 -> 51.8 mm
- net SDA/COPI5: track 42.8 -> 51.8 mm
- net SDA/COPI4: track 42.8 -> 51.8 mm
- net SDA/COPI2: track 42.8 -> 51.8 mm
- net SDA/COPI14: track 42.8 -> 51.8 mm
- net SDA/COPI11: track 42.8 -> 51.8 mm
- net SDA/COPI: track 42.8 -> 51.8 mm
- net SDA/COPI7: track 42.8 -> 51.8 mm
- net SDA/COPI6: track 42.8 -> 51.8 mm
- net SDA/COPI15: track 42.8 -> 51.8 mm
- net SDA/COPI13: track 42.8 -> 51.8 mm
- net SDA/COPI3: track 42.8 -> 51.8 mm
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