File: Hardware/Qwiic_High_Performance_Magnetometer_X01.brd (EAGLE design)
At the start: 25.4 x 25.4 mm, 67 parts, among them J1 Qwiic, J2 Qwiic, U1 MMC5893MA_QFN16

Commit message: Added production files; updated BOM.
Parts:
- removed U$40: (no value), numbers:PCB#163280
- added U$41, U$42: (no value), SER:MMC5983MA0
- moved U$34 13.9 mm to (0.76, 15.0), turned to 90 degrees
- moved U$24 2.03 mm to (12.7, 8.00)
- moved U$1 1.78 mm to (12.4, 9.53)
- moved U$10 0.51 mm to (12.7, 9.53)
- moved U$11 0.25 mm to (12.7, 8.26)
Routing:
- net SDA/COPI: track 42.8 -> 51.8 mm
- net INT: track 14.5 -> 16.5 mm
Changed lines of the file:
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@@
 <setting verticaltext="up"/>
 </settings>
-<grid distance="0.1" unitdist="inch" unit="inch" style="lines" multiple="1" display="yes" altdistance="0.005" altunitdist="inch" altunit="inch"/>
+<grid distance="0.01" unitdist="inch" unit="inch" style="lines" multiple="1" display="yes" altdistance="0.005" altunitdist="inch" altunit="inch"/>
 <layers>
 <layer number="1" name="Top" color="4" fill="1" visible="yes" active="yes"/>
@@
 <wire x1="23.241" y1="5.842" x2="23.749" y2="6.096" width="0.2032" layer="21"/>
 <wire x1="23.749" y1="6.096" x2="23.241" y2="6.35" width="0.2032" layer="21"/>
-<text x="3.302" y="19.812" size="1.27" layer="16" font="vector" ratio="15" rot="MR270">X01</text>
+<text x="2.794" y="19.812" size="1.27" layer="16" font="vector" ratio="15" rot="MR270">X01</text>
 <dimension x1="-1.27" y1="25.4" x2="-1.27" y2="0" x3="-2.54" y3="12.7" textsize="1.778" layer="47" unit="inch"/>
 <dimension x1="0" y1="-1.27" x2="25.4" y2="-1.27" x3="12.7" y3="-3.81" textsize="1.778" layer="47" unit="inch"/>
@@
 <element name="U$7" library="output" package="#INT#7" value="" x="7.62" y="23.749" smashed="yes" rot="R270"/>
 <element name="U$8" library="output" package="PWR9" value="" x="2.54" y="17.78" smashed="yes"/>
-<element name="U$10" library="output" package="HIGH_PERFORMANCE11" value="" x="12.7" y="10.033" smashed="yes"/>
-<element name="U$11" library="output" package="MAGNETOMETER12" value="" x="12.7" y="8.509" smashed="yes"/>
+<element name="U$10" library="output" package="HIGH_PERFORMANCE11" value="" x="12.7" y="9.525" smashed="yes"/>
+<element name="U$11" library="output" package="MAGNETOMETER12" value="" x="12.7" y="8.255" smashed="yes"/>
 <element name="U$12" library="output" package="#3#3V#0" value="" x="15.24" y="23.749" smashed="yes" rot="MR270"/>
 <element name="U$13" library="output" package="#GND#4" value="" x="17.78" y="23.749" smashed="yes" rot="MR270"/>
@@
 <element name="U$27" library="output" package="Z17" value="" x="20.066" y="10.033" smashed="yes" rot="MR0"/>
 <element name="U$17" library="output" package="#GND#4" value="" x="6.35" y="6.096" smashed="yes" rot="R270"/>
-<element name="U$1" library="output" package="HIGH_PERFORMANCE11" value="" x="12.446" y="11.303" smashed="yes" rot="MR0"/>
-<element name="U$24" library="output" package="MAGNETOMETER12" value="" x="12.7" y="10.033" smashed="yes" rot="MR0"/>
+<element name="U$1" library="output" package="HIGH_PERFORMANCE11" value="" x="12.446" y="9.525" smashed="yes" rot="MR0"/>
+<element name="U$24" library="output" package="MAGNETOMETER12" value="" x="12.7" y="8.001" smashed="yes" rot="MR0"/>
 <element name="U$28" library="output" package="#GND#4" value="" x="6.35" y="6.096" smashed="yes" rot="MR270"/>
 <element name="U$29" library="output" package="#3#3V#0" value="" x="8.89" y="6.477" smashed="yes" rot="MR270"/>
@@
 <element name="U$36" library="SparkX" package="SPARKX-TINY" value="SPARKX-LOGO2" x="3.048" y="5.842" smashed="yes"/>
 <element name="U$37" library="SparkX" package="SPARKX-SMALL" value="SPARKX-LOGO3" x="12.954" y="13.97" smashed="yes" rot="MR0"/>
-<element name="U$34" library="output" package="MADE_IN_THE_USA20" value="" x="12.7" y="7.874" smashed="yes" rot="MR0"/>
+<element name="U$34" library="output" package="MADE_IN_THE_USA20" value="" x="0.762" y="14.986" smashed="yes" rot="MR90"/>
 <element name="U$35" library="output" package="#SCL#6" value="" x="12.7" y="23.749" smashed="yes" rot="MR270"/>
 <element name="U$38" library="output" package="#SDA#5" value="" x="10.16" y="23.749" smashed="yes" rot="MR270"/>
 <element name="U$39" library="output" package="Z17" value="" x="20.701" y="4.826" smashed="yes"/>
-<element name="U$40" library="numbers" package="PCB#163280" value="" x="1.016" y="15.748" smashed="yes" rot="MR90"/>
+<element name="U$41" library="SER" package="MMC5983MA0" value="" x="12.7" y="15.494" smashed="yes"/>
+<element name="U$42" library="SER" package="MMC5983MA0" value="" x="12.573" y="11.176" smashed="yes" rot="MR0"/>
 </elements>
 <signals>
@@
 <wire x1="3.564" y1="13.2" x2="3.556" y2="13.208" width="0.508" layer="1"/>
 <via x="3.556" y="13.208" extent="1-16" drill="0.381"/>
-<wire x1="3.556" y1="13.208" x2="6.858" y2="13.208" width="0.508" layer="16"/>
-<wire x1="6.858" y1="13.208" x2="8.89" y2="13.208" width="0.508" layer="16"/>
-<wire x1="8.89" y1="13.208" x2="12.446" y2="13.208" width="0.508" layer="16"/>
+<wire x1="12.446" y1="13.208" x2="8.89" y2="13.208" width="0.508" layer="16"/>
 <wire x1="12.446" y1="13.208" x2="12.7" y2="13.208" width="0.508" layer="16"/>
 <wire x1="12.7" y1="13.208" x2="15.24" y2="13.208" width="0.508" layer="16"/>
@@
 <via x="17.78" y="15.748" extent="1-16" drill="0.3048"/>
 <wire x1="17.78" y1="15.748" x2="15.24" y2="15.748" width="0.508" layer="16"/>
-<wire x1="7.0993" y1="17.78" x2="7.0993" y2="13.4493" width="0.508" layer="16"/>
-<wire x1="7.0993" y1="13.4493" x2="6.858" y2="13.208" width="0.508" layer="16"/>
 <wire x1="12.446" y1="11.202" x2="12.446" y2="12.192" width="0.2032" layer="1"/>
 <via x="12.446" y="12.192" extent="1-16" drill="0.3048"/>
@@
 <wire x1="12.446" y1="12.7" x2="12.446" y2="12.192" width="0.2032" layer="1"/>
 <wire x1="11.682" y1="13.464" x2="12.446" y2="12.7" width="0.2032" layer="1"/>
+<wire x1="8.89" y1="13.208" x2="7.112" y2="13.208" width="0.508" layer="16"/>
+<wire x1="7.112" y1="13.208" x2="3.556" y2="13.208" width="0.508" layer="16"/>
+<wire x1="7.0993" y1="17.78" x2="7.0993" y2="13.2207" width="0.508" layer="16"/>
+<wire x1="7.0993" y1="13.2207" x2="7.112" y2="13.208" width="0.508" layer="16"/>
 </signal>
 <signal name="N$1">
@@
 <contactref element="U1" pad="15"/>
 <contactref element="J3" pad="5"/>
-<via x="10.16" y="15.494" extent="1-16" drill="0.3048"/>
 <wire x1="11.204" y1="12.464" x2="10.396" y2="12.464" width="0.2032" layer="1"/>
 <wire x1="10.396" y1="12.464" x2="10.16" y2="12.7" width="0.2032" layer="1"/>
-<wire x1="10.16" y1="12.7" x2="10.16" y2="15.494" width="0.2032" layer="1"/>
 <wire x1="7.62" y1="21.844" x2="8.128" y2="21.336" width="0.2032" layer="16"/>
 <wire x1="8.128" y1="21.336" x2="9.652" y2="21.336" width="0.2032" layer="16"/>
-<wire x1="9.652" y1="21.336" x2="10.16" y2="20.828" width="0.2032" layer="16"/>
+<wire x1="10.16" y1="20.828" x2="9.652" y2="21.336" width="0.2032" layer="16"/>
 <wire x1="7.62" y1="24.13" x2="7.62" y2="21.844" width="0.2032" layer="16"/>
-<wire x1="10.16" y1="20.828" x2="10.16" y2="15.494" width="0.2032" layer="16"/>
+<wire x1="10.16" y1="12.7" x2="9.398" y2="12.7" width="0.2032" layer="1"/>
+<wire x1="9.398" y1="12.7" x2="8.89" y2="13.208" width="0.2032" layer="1"/>
+<wire x1="8.89" y1="13.208" x2="8.89" y2="14.224" width="0.2032" layer="1"/>
+<via x="8.89" y="14.224" extent="1-16" drill="0.3048"/>
+<wire x1="8.89" y1="14.224" x2="9.652" y2="14.224" width="0.2032" layer="16"/>
+<wire x1="9.652" y1="14.224" x2="10.16" y2="14.732" width="0.2032" layer="16"/>
+<wire x1="10.16" y1="14.732" x2="10.16" y2="20.828" width="0.2032" layer="16"/>
 </signal>
 <signal name="N$2">
@@
 <contactref element="R1" pad="1"/>
 <contactref element="J4" pad="3"/>
-<wire x1="10.16" y1="18.63" x2="10.16" y2="24.13" width="0.2032" layer="1"/>
+<wire x1="10.16" y1="18.63" x2="10.16" y2="20.574" width="0.2032" layer="1"/>
+<wire x1="10.16" y1="20.574" x2="10.16" y2="24.13" width="0.2032" layer="1"/>
 <wire x1="5.08" y1="12.2" x2="9.144" y2="12.2" width="0.2032" layer="1"/>
 <wire x1="11.178" y1="11.938" x2="10.16" y2="11.938" width="0.2032" layer="1"/>
 <wire x1="11.178" y1="11.938" x2="11.204" y2="11.964" width="0.2032" layer="1"/>
-<wire x1="10.16" y1="18.63" x2="9.486" y2="18.63" width="0.2032" layer="1"/>
-<wire x1="9.486" y1="18.63" x2="9.144" y2="18.288" width="0.2032" layer="1"/>
-<wire x1="9.144" y1="18.288" x2="9.144" y2="12.2" width="0.2032" layer="1"/>
-<wire x1="10.16" y1="11.938" x2="10.16" y2="9.144" width="0.2032" layer="1"/>
-<via x="10.16" y="9.144" extent="1-16" drill="0.3048"/>
+<wire x1="10.16" y1="11.938" x2="10.16" y2="10.414" width="0.2032" layer="1"/>
+<via x="10.16" y="10.414" extent="1-16" drill="0.3048"/>
 <via x="16.764" y="12.192" extent="1-16" drill="0.3048"/>
 <wire x1="16.764" y1="12.192" x2="16.764" y2="12.954" width="0.2032" layer="1"/>
@@
 <wire x1="9.144" y1="12.2" x2="9.406" y2="11.938" width="0.2032" layer="1"/>
 <wire x1="9.406" y1="11.938" x2="10.16" y2="11.938" width="0.2032" layer="1"/>
-<wire x1="11.43" y1="1.27" x2="11.43" y2="9.144" width="0.2032" layer="16"/>
-<wire x1="11.43" y1="9.144" x2="11.43" y2="10.668" width="0.2032" layer="16"/>
+<wire x1="11.43" y1="1.27" x2="11.43" y2="10.414" width="0.2032" layer="16"/>
+<wire x1="11.43" y1="10.414" x2="11.43" y2="10.668" width="0.2032" layer="16"/>
 <wire x1="11.43" y1="10.668" x2="11.938" y2="11.176" width="0.2032" layer="16"/>
 <wire x1="11.938" y1="11.176" x2="13.716" y2="11.176" width="0.2032" layer="16"/>
 <wire x1="13.716" y1="11.176" x2="14.732" y2="12.192" width="0.2032" layer="16"/>
 <wire x1="14.732" y1="12.192" x2="16.764" y2="12.192" width="0.2032" layer="16"/>
-<wire x1="10.16" y1="9.144" x2="11.43" y2="9.144" width="0.2032" layer="16"/>
+<wire x1="11.43" y1="10.414" x2="10.16" y2="10.414" width="0.2032" layer="16"/>
+<wire x1="5.08" y1="12.2" x2="3.04" y2="12.2" width="0.2032" layer="1"/>
+<wire x1="3.04" y1="12.2" x2="2.794" y2="12.446" width="0.2032" layer="1"/>
+<wire x1="2.794" y1="12.446" x2="2.794" y2="13.97" width="0.2032" layer="1"/>
+<wire x1="2.794" y1="13.97" x2="3.048" y2="14.224" width="0.2032" layer="1"/>
+<wire x1="3.048" y1="14.224" x2="3.048" y2="20.066" width="0.2032" layer="1"/>
+<wire x1="3.048" y1="20.066" x2="3.556" y2="20.574" width="0.2032" layer="1"/>
+<wire x1="3.556" y1="20.574" x2="10.16" y2="20.574" width="0.2032" layer="1"/>
 </signal>
 <signal name="SCL/SCK">

Commit message: Fixed typo
Parts:
- U1: value MMC5893MA_QFN16 -> MMC5983MA_QFN16
Changed lines of the file:
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@@
 <drawing>
 <settings>
-<setting alwaysvectorfont="yes"/>
+<setting alwaysvectorfont="no"/>
 <setting verticaltext="up"/>
 </settings>
-<grid distance="0.01" unitdist="inch" unit="inch" style="lines" multiple="1" display="yes" altdistance="0.005" altunitdist="inch" altunit="inch"/>
+<grid distance="0.05" unitdist="inch" unit="inch" style="lines" multiple="1" display="yes" altdistance="0.005" altunitdist="inch" altunit="inch"/>
 <layers>
 <layer number="1" name="Top" color="4" fill="1" visible="yes" active="yes"/>
@@
 <attribute name="VALUE" x="8.382" y="17.78" size="0.6096" layer="27" font="vector" ratio="20" rot="R90" align="top-center"/>
 </element>
-<element name="U1" library="SparkFun-Sensors" package="LGA-16-3X3MM-4X4PINS" value="MMC5893MA_QFN16" x="12.7" y="12.7" smashed="yes" rot="R180">
+<element name="U1" library="SparkFun-Sensors" package="LGA-16-3X3MM-4X4PINS" value="MMC5983MA_QFN16" x="12.7" y="12.7" smashed="yes" rot="R180">
 <attribute name="NAME" x="13.335" y="9.525" size="0.6096" layer="25" font="vector" ratio="20" rot="R180"/>
 <attribute name="PROD_ID" value="IC-16314" x="12.7" y="12.7" size="1.778" layer="27" rot="R180" display="off"/>
